File: hardware/kicad/HomeKey-Lock-RevA-PN7161.kicad_pcb (KiCad board)
At the start: 4 copper layers, 150 x 75 mm, 120 parts, among them J1 BATTERY 3S 9.0-12.6V, J2 USB-C USB2, J3 EXT ANT DNP, J4 DS3115 SERVO, Q1 AO4407A, SW1 RESET, SW2 BOOT, SW3 SERVICE, U1 AP63205WU-7 5V, U2 USBLC6-2SC6, U3 AP63203WU-7 3V3, U4 ESP32-C6-MINI-1-N4, U5 PN7161B1HN/C100E, U6 TPS565201DDCR, X1 27.12MHz 10pF

Commit message: Enlarge the NFC coil to 40x65 and retune the match for it
The 40x40 loop was sized by the circuit's position, not by the physics.
Coupling for a loop of radius a at range d peaks at a = d, and at a phone
tap distance of ~30-40 mm through a door leaf the 40x40 coil sat well
below that optimum while 20 mm of board west of it stayed empty.

Growing the loop to 40x65 buys about 1.74 dB of coupling and costs only
two mounting holes: H1 and H3 move from x=4 to x=53. The outline stays
150x75 and no part in the circuit moves.

Parametrise the antenna rather than retype it. AntennaSpec in
design_data.py now derives the spiral, AE1's placement, the copper
keep-out, the B.Cu underpass, the footprint's library name and AE1's
value string from one set of numbers. Four hardcoded keep-out rectangles
and a hardcoded underpass coordinate pair are gone; the underpass pair
was already wrong for any coil but 40x40, which showed up as a dangling
ANT_P track the moment the height changed. Held at height=40 the whole
parametrisation reproduces the previous board byte for byte.

Retune the matching network, which is the part that would have shipped
broken. The taller coil is 1.979 uH against 1.491, so the Rev A 68p/100p
pair resonates it at 12.11 MHz -- two bandwidths low. Both capacitors
scale by 0.75 to 51p/75p, which keeps Cp/Cs at 1.471 exactly as before,
so the impedance the PN7161 driver sees barely moves (12.75 -> 13.83 ohm,
1.7 degrees). C29/C30 become C519494 and C31/C32 become C519496, both
YAGEO NP0 +-1% 50V 0603, verified against LCSC's own product pages.

Commit the ngspice deck. PREFAB_REVIEW_ACTIONS.md quoted simulation
results the repo could not reproduce; design/sim/nfc_match.cir and
sweep.py now regenerate every number in that section. The deck lands
Rev A at 13.805 MHz rather than the 13.601 recorded earlier -- it
terminates the RX taps, which that run evidently did not -- so the
section now reports offsets against where Rev A itself lands instead of
against 13.560 absol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
Parts:
- AE1: value 40x40mm 4-turn PCB antenna -> 40x65mm 4-turn PCB antenna; footprint HomeKey_RevA:NFC_Antenna_40x40_4T -> HomeKey_RevA:NFC_Antenna_40x65_4T
- C29, C30: value 68pF C0G 2% -> 51pF NP0 1%
- C31, C32: value 100pF C0G 2% -> 75pF NP0 1%
- moved H1 49.0 mm to (53.0, 4.00)
- moved H3 49.0 mm to (53.0, 71.0)
Routing:
- net ANT_P: track 19.8 -> 31.9 mm
Changed lines of the file:
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@@
       (effects (font (size 1 1) (thickness 0.15)))
     )
-    (fp_text value "68pF C0G 2%" (at 0 1.43 180) (layer "F.Fab") hide
+    (fp_text value "51pF NP0 1%" (at 0 1.43 180) (layer "F.Fab") hide
       (effects (font (size 1 1) (thickness 0.15)))
     )
@@
       (effects (font (size 1 1) (thickness 0.15)))
     )
-    (fp_text value "68pF C0G 2%" (at 0 1.43 180) (layer "F.Fab") hide
+    (fp_text value "51pF NP0 1%" (at 0 1.43 180) (layer "F.Fab") hide
       (effects (font (size 1 1) (thickness 0.15)))
     )
@@
       (effects (font (size 1 1) (thickness 0.15)))
     )
-    (fp_text value "100pF C0G 2%" (at 0 1.43 90) (layer "F.Fab") hide
+    (fp_text value "75pF NP0 1%" (at 0 1.43 90) (layer "F.Fab") hide
       (effects (font (size 1 1) (thickness 0.15)))
     )
@@
       (effects (font (size 1 1) (thickness 0.15)))
     )
-    (fp_text value "100pF C0G 2%" (at 0 1.43 90) (layer "F.Fab") hide
+    (fp_text value "75pF NP0 1%" (at 0 1.43 90) (layer "F.Fab") hide
       (effects (font (size 1 1) (thickness 0.15)))
     )
@@
     )
   )
-  (footprint "HomeKey_RevA:NFC_Antenna_40x40_4T" (version 20221018) (generator pcbnew) (layer "F.Cu")
+  (footprint "HomeKey_RevA:NFC_Antenna_40x65_4T" (version 20221018) (generator pcbnew) (layer "F.Cu")
     (at 48 37.5 0)
     (path "/generated/AE1")
     (attr board_only exclude_from_pos_files exclude_from_bom)
     (net_tie_pad_groups "1,2")
-    (fp_text reference "AE1" (at -23 -23 0) (layer "F.SilkS")
+    (fp_text reference "AE1" (at -23 -35.5 0) (layer "F.SilkS")
       (effects (font (size 1 1) (thickness 0.15)))
     )
-    (fp_text value "40x40mm 4-turn PCB antenna" (at -23 23 0) (layer "F.Fab") hide
+    (fp_text value "40x65mm 4-turn PCB antenna" (at -23 35.5 0) (layer "F.Fab") hide
       (effects (font (size 1 1) (thickness 0.15)))
     )
     (fp_line (start 0 -2.5) (end -3 -2.5) (layer "F.Cu") (stroke (width 0.4) (type solid)))
-    (fp_line (start -3 -2.5) (end -3 -20) (layer "F.Cu") (stroke (width 0.4) (type solid)))
-    (fp_line (start -3 -20) (end -43 -20) (layer "F.Cu") (stroke (width 0.4) (type solid)))
-    (fp_line (start -43 -20) (end -43 20) (layer "F.Cu") (stroke (width 0.4) (type solid)))
-    (fp_line (start -43 20) (end -3.7 20) (layer "F.Cu") (stroke (width 0.4) (type solid)))
-    (fp_line (start -3.7 20) (end -3.7 -19.3) (layer "F.Cu") (stroke (width 0.4) (type solid)))
-    (fp_line (start -3.7 -19.3) (end -42.3 -19.3) (layer "F.Cu") (stroke (width 0.4) (type solid)))
-    (fp_line (start -42.3 -19.3) (end -42.3 19.3) (layer "F.Cu") (stroke (width 0.4) (type solid)))
-    (fp_line (start -42.3 19.3) (end -4.4 19.3) (layer "F.Cu") (stroke (width 0.4) (type solid)))
-    (fp_line (start -4.4 19.3) (end -4.4 -18.6) (layer "F.Cu") (stroke (width 0.4) (type solid)))
-    (fp_line (start -4.4 -18.6) (end -41.6 -18.6) (layer "F.Cu") (stroke (width 0.4) (type solid)))
-    (fp_line (start -41.6 -18.6) (end -41.6 18.6) (layer "F.Cu") (stroke (width 0.4) (type solid)))
-    (fp_line (start -41.6 18.6) (end -5.1 18.6) (layer "F.Cu") (stroke (width 0.4) (type solid)))
-    (fp_line (start -5.1 18.6) (end -5.1 -17.9) (layer "F.Cu") (stroke (width 0.4) (type solid)))
-    (fp_line (start -5.1 -17.9) (end -40.9 -17.9) (layer "F.Cu") (stroke (width 0.4) (type solid)))
-    (fp_line (start -40.9 -17.9) (end -40.9 17.9) (layer "F.Cu") (stroke (width 0.4) (type solid)))
-    (fp_line (start -40.9 17.9) (end -5.8 17.9) (layer "F.Cu") (stroke (width 0.4) (type solid)))
-    (fp_line (start -5.8 17.9) (end 0 2.5) (layer "B.Cu") (stroke (width 0.4) (type solid)))
+    (fp_line (start -3 -2.5) (end -3 -32.5) (layer "F.Cu") (stroke (width 0.4) (type solid)))
+    (fp_line (start -3 -32.5) (end -43 -32.5) (layer "F.Cu") (stroke (width 0.4) (type solid)))
+    (fp_line (start -43 -32.5) (end -43 32.5) (layer "F.Cu") (stroke (width 0.4) (type solid)))
+    (fp_line (start -43 32.5) (end -3.7 32.5) (layer "F.Cu") (stroke (width 0.4) (type solid)))
+    (fp_line (start -3.7 32.5) (end -3.7 -31.8) (layer "F.Cu") (stroke (width 0.4) (type solid)))
+    (fp_line (start -3.7 -31.8) (end -42.3 -31.8) (layer "F.Cu") (stroke (width 0.4) (type solid)))
+    (fp_line (start -42.3 -31.8) (end -42.3 31.8) (layer "F.Cu") (stroke (width 0.4) (type solid)))
+    (fp_line (start -42.3 31.8) (end -4.4 31.8) (layer "F.Cu") (stroke (width 0.4) (type solid)))
+    (fp_line (start -4.4 31.8) (end -4.4 -31.1) (layer "F.Cu") (stroke (width 0.4) (type solid)))
+    (fp_line (start -4.4 -31.1) (end -41.6 -31.1) (layer "F.Cu") (stroke (width 0.4) (type solid)))
+    (fp_line (start -41.6 -31.1) (end -41.6 31.1) (layer "F.Cu") (stroke (width 0.4) (type solid)))
+    (fp_line (start -41.6 31.1) (end -5.1 31.1) (layer "F.Cu") (stroke (width 0.4) (type solid)))
+    (fp_line (start -5.1 31.1) (end -5.1 -30.4) (layer "F.Cu") (stroke (width 0.4) (type solid)))
+    (fp_line (start -5.1 -30.4) (end -40.9 -30.4) (layer "F.Cu") (stroke (width 0.4) (type solid)))
+    (fp_line (start -40.9 -30.4) (end -40.9 30.4) (layer "F.Cu") (stroke (width 0.4) (type solid)))
+    (fp_line (start -40.9 30.4) (end -5.8 30.4) (layer "F.Cu") (stroke (width 0.4) (type solid)))
+    (fp_line (start -5.8 30.4) (end 0 2.5) (layer "B.Cu") (stroke (width 0.4) (type solid)))
     (pad "1" smd rect (at 0 -2.5) (size 1.2 1.2) (layers "F.Cu" "F.Paste" "F.Mask")
       (net 3 "ANT_N"))
-    (pad "2" thru_hole circle (at -5.8 17.9) (size 1.2 1.2) (drill 0.5) (layers *.Cu *.Mask)
+    (pad "2" thru_hole circle (at -5.8 30.4) (size 1.2 1.2) (drill 0.5) (layers *.Cu *.Mask)
       (net 4 "ANT_P"))
     (pad "2" thru_hole circle (at 0 2.5) (size 1.2 1.2) (drill 0.5) (layers *.Cu *.Mask)
@@
   )
   (footprint "HomeKey_RevA:MountingHole_3.2mm_M3" (version 20211014) (generator pcbnew) (layer "F.Cu")
-    (at 4 4 0)
+    (at 53 4 0)
     (descr "Mounting Hole 3.2mm, no annular, M3")
     (tags "mounting hole 3.2mm no annular m3")
@@
   )
   (footprint "HomeKey_RevA:MountingHole_3.2mm_M3" (version 20211014) (generator pcbnew) (layer "F.Cu")
-    (at 4 71 0)
+    (at 53 71 0)
     (descr "Mounting Hole 3.2mm, no annular, M3")
     (tags "mounting hole 3.2mm no annular m3")
@@
   (segment (start 120.4 20.5) (end 127.6 20.5) (width 0.25) (layer "F.Cu") (net 9))
   (segment (start 132.4 20.5) (end 139.6 20.5) (width 0.25) (layer "F.Cu") (net 45))
-  (segment (start 42.2 55.4) (end 48.0 40.0) (width 0.4) (layer "B.Cu") (net 4))
+  (segment (start 42.2 67.9) (end 48.0 40.0) (width 0.4) (layer "B.Cu") (net 4))
   (segment (start 86.0 32.775) (end 88.5 32.775) (width 0.5) (layer "F.Cu") (net 57))
   (segment (start 100.0 36.7) (end 100.95 36.7) (width 0.2) (layer "F.Cu") (net 57))
@@
     (placement (enabled no) (sheetname ""))
     (fill (thermal_gap 0.508) (thermal_bridge_width 0.508) (island_removal_mode 0))
-    (polygon (pts (xy 48.5 59.0) (xy 0.0 59.0) (xy 0.0 16.0) (xy 48.5 16.0)))
+    (polygon (pts (xy 48.5 71.5) (xy 0.0 71.5) (xy 0.0 3.5) (xy 48.5 3.5)))
   )
   (zone
